Commit message: feat: stabilize robot with symmetric ball casters

File: src/symbotic_description/urdf/differential_drive.urdf.xacro (robot description, xacro)
@@ -9,4 +9,5 @@
   <xacro:property name="geometry" value="${config['robot']['geometry']}"/>
   <xacro:property name="dynamics" value="${config['robot']['dynamics']}"/>
+  <xacro:property name="limits" value="${config['robot']['limits']}"/>
   <xacro:property name="track_width" value="${geometry['track_width']}"/>
   <xacro:property name="wheelbase" value="${geometry['wheelbase']}"/>
@@ -60,4 +61,11 @@
     </inertial>
   </xacro:macro>
+  <!-- Massless ground-projected root frame keeps KDL and TF trees well formed. -->
+  <link name="base_footprint"/>
+  <joint name="base_footprint_joint" type="fixed">
+    <parent link="base_footprint"/>
+    <child link="base_link"/>
+    <origin xyz="0 0 ${base_height}" rpy="0 0 0"/>
+  </joint>
   <link name="base_link">
     <xacro:box_inertia
@@ -110,26 +118,30 @@
   <xacro:drive_wheel name="left" y_sign="1"/>
   <xacro:drive_wheel name="right" y_sign="-1"/>
-  <!-- +X is the front of the robot. The ball caster is centered at the rear. -->
-  <link name="rear_ball_caster">
-    <xacro:sphere_inertia mass="${caster_mass}" radius="${caster_radius}"/>
-    <visual>
-      <geometry>
-        <sphere radius="${caster_radius}"/>
-      </geometry>
-      <material name="caster_material">
-        <color rgba="0.12 0.12 0.12 1.0"/>
-      </material>
-    </visual>
-    <collision>
-      <geometry>
-        <sphere radius="${caster_radius}"/>
-      </geometry>
-    </collision>
-  </link>
-  <joint name="rear_ball_caster_joint" type="fixed">
-    <parent link="base_link"/>
-    <child link="rear_ball_caster"/>
-    <origin xyz="${-wheelbase} 0 ${caster_z}" rpy="0 0 0"/>
-  </joint>
+  <!-- +X is the front. Symmetric ball casters prevent pitch during braking. -->
+  <xacro:macro name="ball_caster" params="name x">
+    <link name="${name}_ball_caster">
+      <xacro:sphere_inertia mass="${caster_mass}" radius="${caster_radius}"/>
+      <visual>
+        <geometry>
+          <sphere radius="${caster_radius}"/>
+        </geometry>
+        <material name="caster_material">
+          <color rgba="0.12 0.12 0.12 1.0"/>
+        </material>
+      </visual>
+      <collision>
+        <geometry>
+          <sphere radius="${caster_radius}"/>
+        </geometry>
+      </collision>
+    </link>
+    <joint name="${name}_ball_caster_joint" type="fixed">
+      <parent link="base_link"/>
+      <child link="${name}_ball_caster"/>
+      <origin xyz="${x} 0 ${caster_z}" rpy="0 0 0"/>
+    </joint>
+  </xacro:macro>
+  <xacro:ball_caster name="front" x="${wheelbase}"/>
+  <xacro:ball_caster name="rear" x="${-wheelbase}"/>
   <gazebo reference="base_link">
     <mu1>0.8</mu1>
@@ -144,7 +156,35 @@
     <mu2>1.5</mu2>
   </gazebo>
+  <gazebo reference="front_ball_caster">
+    <mu1>0.2</mu1>
+    <mu2>0.2</mu2>
+  </gazebo>
   <gazebo reference="rear_ball_caster">
     <mu1>0.2</mu1>
     <mu2>0.2</mu2>
   </gazebo>
+  <gazebo>
+    <plugin filename="gz-sim-diff-drive-system" name="gz::sim::systems::DiffDrive">
+      <left_joint>left_wheel_joint</left_joint>
+      <right_joint>right_wheel_joint</right_joint>
+      <wheel_separation>${track_width}</wheel_separation>
+      <wheel_radius>${wheel_radius}</wheel_radius>
+      <topic>/cmd_vel</topic>
+      <odom_topic>/odom</odom_topic>
+      <tf_topic>/tf</tf_topic>
+      <child_frame_id>base_footprint</child_frame_id>
+      <odom_publish_frequency>50</odom_publish_frequency>
+      <max_linear_velocity>${limits['max_linear_velocity']}</max_linear_velocity>
+      <min_linear_velocity>${-limits['max_linear_velocity']}</min_linear_velocity>
+      <max_angular_velocity>${limits['max_angular_velocity']}</max_angular_velocity>
+      <min_angular_velocity>${-limits['max_angular_velocity']}</min_angular_velocity>
+      <max_linear_acceleration>${limits['max_linear_acceleration']}</max_linear_acceleration>
+      <min_linear_acceleration>${-limits['max_linear_deceleration']}</min_linear_acceleration>
+      <max_angular_acceleration>${limits['max_angular_acceleration']}</max_angular_acceleration>
+      <min_angular_acceleration>${-limits['max_angular_acceleration']}</min_angular_acceleration>
+    </plugin>
+    <plugin
+      filename="gz-sim-joint-state-publisher-system"
+      name="gz::sim::systems::JointStatePublisher"/>
+  </gazebo>
 </robot>

File: src/symbotic_description/urdf/naked/symbotic_diff_drive.urdf (robot description, URDF)
Before this commit: robot symbotic_diff_drive, 4 links, 3 joints
Links:
- added link base_footprint
- added link front_ball_caster, mass 0.25; collision sphere radius=0.06; visual sphere radius=0.06
Joints:
- added joint base_footprint_joint: type fixed, parent base_footprint, child base_link, origin xyz=0 0 0.295 rpy=0 0 0
- added joint front_ball_caster_joint: type fixed, parent base_link, child front_ball_caster, origin xyz=0.3 0 -0.235 rpy=0 0 0

Commit message: feat: add configurable robot parameters

File: src/symbotic_description/urdf/differential_drive.urdf.xacro (robot description, xacro)
@@ -3,11 +3,11 @@
   <xacro:arg
     name="config_file"
-    default="$(find symbotic_description)/config/robot.yaml"/>
-  <!-- Keep all dimensions and masses in robot.yaml. -->
+    default="$(find symbotic_description)/config/robot_params.yaml"/>
+  <!-- Keep geometry, dynamics and limits in robot_params.yaml. -->
   <xacro:property name="config_file" value="$(arg config_file)"/>
   <xacro:property name="config" value="${xacro.load_yaml(config_file)}"/>
   <xacro:property name="geometry" value="${config['robot']['geometry']}"/>
   <xacro:property name="dynamics" value="${config['robot']['dynamics']}"/>
-  <xacro:property name="limits" value="${config['robot']['limits']}"/>
+  <xacro:property name="controller" value="${config['robot']['controller']}"/>
   <xacro:property name="track_width" value="${geometry['track_width']}"/>
   <xacro:property name="wheelbase" value="${geometry['wheelbase']}"/>
@@ -175,12 +175,12 @@
       <child_frame_id>base_footprint</child_frame_id>
       <odom_publish_frequency>50</odom_publish_frequency>
-      <max_linear_velocity>${limits['max_linear_velocity']}</max_linear_velocity>
-      <min_linear_velocity>${-limits['max_linear_velocity']}</min_linear_velocity>
-      <max_angular_velocity>${limits['max_angular_velocity']}</max_angular_velocity>
-      <min_angular_velocity>${-limits['max_angular_velocity']}</min_angular_velocity>
-      <max_linear_acceleration>${limits['max_linear_acceleration']}</max_linear_acceleration>
-      <min_linear_acceleration>${-limits['max_linear_deceleration']}</min_linear_acceleration>
-      <max_angular_acceleration>${limits['max_angular_acceleration']}</max_angular_acceleration>
-      <min_angular_acceleration>${-limits['max_angular_acceleration']}</min_angular_acceleration>
+      <max_linear_velocity>${controller['max_velocity']}</max_linear_velocity>
+      <min_linear_velocity>${-controller['max_velocity']}</min_linear_velocity>
+      <max_angular_velocity>${controller['max_angular_velocity']}</max_angular_velocity>
+      <min_angular_velocity>${-controller['max_angular_velocity']}</min_angular_velocity>
+      <max_linear_acceleration>${controller['max_acceleration']}</max_linear_acceleration>
+      <min_linear_acceleration>${-controller['max_deceleration']}</min_linear_acceleration>
+      <max_angular_acceleration>${controller['max_angular_acceleration']}</max_angular_acceleration>
+      <min_angular_acceleration>${-controller['max_angular_deceleration']}</min_angular_acceleration>
     </plugin>
     <plugin
